Commit message: lai loi

File: description/robot.urdf.xacro (robot description, xacro)
@@ -1,3 +1,4 @@
 <?xml version="1.0"?>
 <robot xmlns:xacro="http://www.ros.org/wiki/xacro"  name="robot">
+<xacro:include filename="robot_core.xacro"/>
 </robot>

File: description/robot_core.xacro (robot description, xacro)
@@ -22,5 +22,5 @@
 <link name="chassis">
 <visual>
-    <oringin xyz="0.15 0 0.075"/>
+    <origin xyz="0.15 0 0.075"/>
         <geometry>
             <box size="0.3 0.3 0.15"/>
